Commit message: Package name for mesh corrected.

File: urdf/bike.urdf (robot description, URDF)
Before this commit: robot bike, 7 links, 6 joints
Links:
- link robot/backWheelLink: geometry collision mesh filename=package://mobro_sim/urdf/files/wheel_scaled.stl; visual mesh filename=package://mobro_sim/urdf/files/wheel_scaled.stl
- link robot/carrot: geometry visual mesh filename=package://mobro_sim/urdf/carrot/carrot.dae scale=0.003 0.003 0.003
- link robot/frameLink: geometry collision mesh filename=package://mobro_sim/urdf/files/frame_scaled_left.stl; collision mesh filename=package://mobro_sim/urdf/files/frame_scaled_right.stl
- link robot/frontWheelLink: geometry collision mesh filename=package://mobro_sim/urdf/files/wheel_scaled.stl; visual mesh filename=package://mobro_sim/urdf/files/wheel_scaled.stl
- link robot/handlebarLink: geometry collision mesh filename=package://mobro_sim/urdf/files/handlebar_scaled.stl; visual mesh filename=package://mobro_sim/urdf/files/handlebar_scaled.stl
